File: Kicad/noeud_senseur.kicad_pcb (KiCad board)
At the start: 2 copper layers, 100 x 70 mm, 92 parts, among them Q1 DMG1012UW, Q2 DMG1012UW, Q3 LP0701_SGD, Q4 MMBT3904, Q5 MMBT3904, Q6 MMBT3904, U2 DS18B20, U4 SN65HVD232Q, U5 MCP2515, U6 AT24LC256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

Commit message: Mise a jour du 6 juillet 2017
Parts:
- added JP1: Jumper, Pin_Headers:Pin_Header_Straight_1x02_Pitch2.54mm, F.Cu at (124.6, 101.8)
- added R23: 10k, Resistors_SMD:R_0805_HandSoldering, B.Cu at (158.5, 110.2)
- C12, C13, C14: value 0.1uF -> 1uF
- VT-1: value BARREL_JACK -> Barrel_Jack
- moved R1 0.53 mm to (145.5, 94.5)
- moved C11 0.45 mm to (135.0, 126.5)
- moved R18 0.39 mm to (120.1, 128.1)
- moved R21 0.39 mm to (124.5, 128.1)
- moved R19 0.06 mm to (120.1, 123.0)
- turned C1 to 0 degrees
Connections:
- C1 pad 1: +3V3 -> GND
- C1 pad 2: GND -> +3V3
- L10 pad 2: /A1 -> GND
- L3 pad 2: +3V3 -> /A0
- L4 pad 2: /A0 -> GND
- L9 pad 2: +3V3 -> /A1
- R13 pad 1: /A1 -> +3V3
- R13 pad 2: GND -> /A1
- R7 pad 1: /A0 -> +3V3
- R7 pad 2: GND -> /A0
Routing:
- net /MCP2515_INT: track 14.9 -> 35.6 mm, vias 0 -> 2
- net /I2C/INT_SQW: track 31.7 -> 41.1 mm
- net Net-(R23-Pad2): track 0.00 -> 4.99 mm, vias 0 -> 1
- net GND: track 529.7 -> 526.0 mm, vias 27 -> 30
- net /A1: track 56.8 -> 54.0 mm
- net +3V3: track 408.3 -> 406.2 mm, vias 10 -> 11
- net /A0: track 54.5 -> 52.5 mm
- net /A2: track 96.9 -> 96.4 mm
Other:
- board text added: "+"
- board text added: "-"
- board text added: "3V3"
- board text added: "CANH"
- board text added: "CANL"
- board text added: "Cob St-Ambroise CompostNode V. 1.1 Juin 2017"
- board text added: "GND"
- board text added: "IO"
- board text added: "RX"
- board text added: "SCL"
- board text added: "SDA"
- board text added: "TX"
- board text added: "X"
- board text removed: "Cob St-Ambroise CompostNode V. 1.00 Avril 2017"
