File: Kicad/Connect.sch (KiCad schematic (older format))
At the start: 43 parts, among them Q4 MMBT3904, Q5 MMBT3904, Q6 MMBT3904

Commit message: Mise a jour du 6 juillet 2017
Parts:
- C13, C14: value 0.1uF -> 1uF
Connections:
- net +3V3: now also R13.1, R7.1; no longer L3.2, L9.2
- net GND: now also L10.2, L4.2; no longer R13.2, R7.2
- net NTC_1: now also L3.2, R7.2; no longer L4.2, R7.1
- net NTC_2: now also L9.2, R13.2; no longer L10.2, R13.1
Other:
- moved on the sheet: L10, L3, L4, L9, NTC-1, NTC-2, R13, R7

Commit message: Recompilation des applications.
Parts:
- C11: symbol CP -> noeud_senseur-rescue:CP-RESCUE-noeud_senseur
- C13, C14: symbol C_Small -> noeud_senseur-rescue:C_Small-RESCUE-noeud_senseur
- CAN-1, CAN-2, NTC-1, NTC-2, SSR-1, SSR-2: symbol CONN_01X02 -> noeud_senseur-rescue:CONN_01X02-RESCUE-noeud_senseur
- CNJ-1: symbol CAN_NODE_JUNCTION -> jfng:CAN_NODE_JUNCTION
- I2C-1, PWR-1, TM-1: symbol CONN_01X04 -> noeud_senseur-rescue:CONN_01X04-RESCUE-noeud_senseur
- L1, L10, L11, L12, L13, L14, L15, L16, L2, L3, L4, L5, L6, L7, L8, L9: symbol L_Core_Ferrite -> noeud_senseur-rescue:L_Core_Ferrite-RESCUE-noeud_senseur
- OW-1, SER-1: symbol CONN_01X03 -> noeud_senseur-rescue:CONN_01X03-RESCUE-noeud_senseur
- Q4, Q5, Q6: symbol MMBT3904 -> noeud_senseur-rescue:MMBT3904-RESCUE-noeud_senseur
- R10, R11, R12, R13, R14, R22, R7, R8, R9: symbol R -> noeud_senseur-rescue:R-RESCUE-noeud_senseur
