File: Kicad/I2C.sch (KiCad schematic (older format))
At the start: 5 parts, among them U6 AT24LC256, U7 DS3231

Commit message: Recompilation des applications.
Parts:
- BT1: symbol Battery_Cell -> noeud_senseur-rescue:Battery_Cell-RESCUE-noeud_senseur
- C7, C8: symbol C_Small -> noeud_senseur-rescue:C_Small-RESCUE-noeud_senseur
- U6: symbol AT24LC256 -> jfng:AT24LC256
- U7: symbol DS3231 -> jfng:DS3231
Changed lines of the file:
@@
-EESchema Schematic File Version 2
-LIBS:noeud_senseur-rescue
-LIBS:power
-LIBS:device
-LIBS:transistors
-LIBS:conn
-LIBS:linear
-LIBS:regul
-LIBS:74xx
-LIBS:cmos4000
-LIBS:adc-dac
-LIBS:memory
-LIBS:xilinx
-LIBS:microcontrollers
-LIBS:dsp
-LIBS:microchip
-LIBS:analog_switches
-LIBS:motorola
-LIBS:texas
-LIBS:intel
-LIBS:audio
-LIBS:interface
-LIBS:digital-audio
-LIBS:philips
-LIBS:display
-LIBS:cypress
-LIBS:siliconi
-LIBS:opto
-LIBS:atmel
-LIBS:contrib
-LIBS:valves
-LIBS:jfng
+EESchema Schematic File Version 4
 LIBS:noeud_senseur-cache
 EELAYER 26 0
@@
 $EndDescr
 $Comp
-L AT24LC256 U6
+L jfng:AT24LC256 U6
 U 1 1 58C0D972
 P 4300 5325
@@
 $EndComp
 $Comp
-L GND #PWR24
+L noeud_senseur-rescue:GND-RESCUE-noeud_senseur #PWR24
 U 1 1 58C0D979
 P 4300 5800
@@
 $EndComp
 $Comp
-L +3.3V #PWR23
+L noeud_senseur-rescue:+3.3V-RESCUE-noeud_senseur #PWR23
 U 1 1 58C0D97F
 P 4300 4625
@@
 SDA
 $Comp
-L C_Small C7
+L noeud_senseur-rescue:C_Small-RESCUE-noeud_senseur C7
 U 1 1 58C0D987
 P 5150 4825
@@
 $EndComp
 $Comp
-L GND #PWR27
+L noeud_senseur-rescue:GND-RESCUE-noeud_senseur #PWR27
 U 1 1 58C0D98E
 P 5150 4950
@@
 	4300 4625 4300 4975
 $Comp
-L DS3231 U7
+L jfng:DS3231 U7
 U 1 1 58C1AA49
 P 4675 2900
@@
 $EndComp
 $Comp
-L +3.3V #PWR25
+L noeud_senseur-rescue:+3.3V-RESCUE-noeud_senseur #PWR25
 U 1 1 58C1AA50
 P 4675 1925
@@
 $EndComp
 $Comp
-L GND #PWR26
+L noeud_senseur-rescue:GND-RESCUE-noeud_senseur #PWR26
 U 1 1 58C1AA56
 P 4675 3700
@@
 SDA
 $Comp
-L Battery_Cell BT1
+L noeud_senseur-rescue:Battery_Cell-RESCUE-noeud_senseur BT1
 U 1 1 58C1AA5E
 P 3950 3375
@@
 NoConn ~ 5175 3100
 $Comp
-L PWR_FLAG #FLG3
+L noeud_senseur-rescue:PWR_FLAG-RESCUE-noeud_senseur #FLG3
 U 1 1 58C1AA68
 P 3950 3075
@@
 $EndComp
 $Comp
-L C_Small C8
+L noeud_senseur-rescue:C_Small-RESCUE-noeud_senseur C8
 U 1 1 58C1AA6E
 P 5325 2275
@@
 $EndComp
 $Comp
-L GND #PWR28
+L noeud_senseur-rescue:GND-RESCUE-noeud_senseur #PWR28
 U 1 1 58C1AA75
 P 5325 2425
