File: Kicad/PowerMonitoring.sch (KiCad schematic (older format))
At the start: 11 parts

Commit message: Mise a jour du 6 juillet 2017
Parts:
- removed VT-1: BARREL_JACK, Connectors_Molex:Molex_KK-6410-03_03x2.54mm_Straight, symbol BARREL_JACK
- added VT-1: Barrel_Jack, Connectors_Molex:Molex_KK-6410-03_03x2.54mm_Straight, symbol Barrel_Jack
Connections:
- net at C10.1, R19.2, R20.2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: now also VT-1.2, VT-1.3
- net at R18.2: now also VT-1.1
Changed lines of the file:
@@
 EESchema Schematic File Version 2
+LIBS:noeud_senseur-rescue
 LIBS:power
 LIBS:device
@@
 EELAYER 26 0
 EELAYER END
-$Descr A4 11693 8268
+$Descr USLetter 11000 8500
 encoding utf-8
 Sheet 5 5
-Title ""
-Date ""
-Rev ""
+Title "Power Monitoring"
+Date "2017-06-06"
+Rev "1.1"
 Comp ""
 Comment1 ""
@@
 $EndComp
 $Comp
-L +3.3V #PWR054
+L +3.3V #PWR52
 U 1 1 58DBFD32
 P 2950 1375
-F 0 "#PWR054" H 2950 1225 50  0001 C CNN
+F 0 "#PWR52" H 2950 1225 50  0001 C CNN
 F 1 "+3.3V" H 2965 1548 50  0000 C CNN
 F 2 "" H 2950 1375 50  0001 C CNN
@@
 $EndComp
 $Comp
-L GND #PWR055
+L GND #PWR51
 U 1 1 58DBFD9A
 P 2575 2600
-F 0 "#PWR055" H 2575 2350 50  0001 C CNN
+F 0 "#PWR51" H 2575 2350 50  0001 C CNN
 F 1 "GND" H 2580 2427 50  0000 C CNN
 F 2 "" H 2575 2600 50  0001 C CNN
@@
 Connection ~ 2950 2050
 $Comp
-L GND #PWR056
+L GND #PWR53
 U 1 1 58DC135A
 P 2950 2600
-F 0 "#PWR056" H 2950 2350 50  0001 C CNN
+F 0 "#PWR53" H 2950 2350 50  0001 C CNN
 F 1 "GND" H 2955 2427 50  0000 C CNN
 F 2 "" H 2950 2600 50  0001 C CNN
@@
 $EndComp
 $Comp
-L +3.3V #PWR057
+L +3.3V #PWR55
 U 1 1 58DC40BE
 P 6475 1375
-F 0 "#PWR057" H 6475 1225 50  0001 C CNN
+F 0 "#PWR55" H 6475 1225 50  0001 C CNN
 F 1 "+3.3V" H 6490 1548 50  0000 C CNN
 F 2 "" H 6475 1375 50  0001 C CNN
@@
 $EndComp
 $Comp
-L GND #PWR058
+L GND #PWR54
 U 1 1 58DC40C4
 P 6100 2600
-F 0 "#PWR058" H 6100 2350 50  0001 C CNN
+F 0 "#PWR54" H 6100 2350 50  0001 C CNN
 F 1 "GND" H 6105 2427 50  0000 C CNN
 F 2 "" H 6100 2600 50  0001 C CNN
@@
 Connection ~ 6475 2050
 $Comp
-L GND #PWR059
+L GND #PWR56
 U 1 1 58DC40D8
 P 6475 2600
-F 0 "#PWR059" H 6475 2350 50  0001 C CNN
+F 0 "#PWR56" H 6475 2350 50  0001 C CNN
 F 1 "GND" H 6480 2427 50  0000 C CNN
 F 2 "" H 6475 2600 50  0001 C CNN
@@
 Wire Wire Line
 	1800 1850 1575 1850
-$Comp
-L BARREL_JACK VT-1
-U 1 1 58E22486
-P 4700 1650
-F 0 "VT-1" H 4681 1975 50  0000 C CNN
-F 1 "BARREL_JACK" H 4681 1884 50  0000 C CNN
-F 2 "Connectors_Molex:Molex_KK-6410-03_03x2.54mm_Straight" H 4700 1650 50  0001 C CNN
-F 3 "" H 4700 1650 50  0001 C CNN
-	1    4700 1650
-	1    0    0    -1
-$EndComp
 Wire Wire Line
 	5175 2050 5175 1650
@@
 Connection ~ 5175 1750
 NoConn ~ 1575 1650
+$Comp
+L Barrel_Jack VT-1
+U 1 1 5939738C
+P 4700 1650
+F 0 "VT-1" H 4778 1975 50  0000 C CNN
+F 1 "Barrel_Jack" H 4778 1884 50  0000 C CNN
+F 2 "Connectors_Molex:Molex_KK-6410-03_03x2.54mm_Straight" H 4750 1610 50  0001 C CNN
+F 3 "" H 4750 1610 50  0001 C CNN
+	1    4700 1650
+	1    0    0    -1
+$EndComp
 $EndSCHEMATC

Commit message: Recompilation des applications.
Parts:
- C10, C9: symbol CP -> noeud_senseur-rescue:CP-RESCUE-noeud_senseur
- CT-1: symbol JACK_TRS_3PINS -> jfng:JACK_TRS_3PINS
- R15, R16, R17, R18, R19, R20, R21: symbol R -> noeud_senseur-rescue:R-RESCUE-noeud_senseur
- VT-1: symbol Barrel_Jack -> jfng:Barrel_Jack
Changed lines of the file:
@@
-EESchema Schematic File Version 2
-LIBS:noeud_senseur-rescue
-LIBS:power
-LIBS:device
-LIBS:transistors
-LIBS:conn
-LIBS:linear
-LIBS:regul
-LIBS:74xx
-LIBS:cmos4000
-LIBS:adc-dac
-LIBS:memory
-LIBS:xilinx
-LIBS:microcontrollers
-LIBS:dsp
-LIBS:microchip
-LIBS:analog_switches
-LIBS:motorola
-LIBS:texas
-LIBS:intel
-LIBS:audio
-LIBS:interface
-LIBS:digital-audio
-LIBS:philips
-LIBS:display
-LIBS:cypress
-LIBS:siliconi
-LIBS:opto
-LIBS:atmel
-LIBS:contrib
-LIBS:valves
-LIBS:jfng
+EESchema Schematic File Version 4
 LIBS:noeud_senseur-cache
 EELAYER 26 0
@@
 $EndDescr
 $Comp
-L R R17
+L noeud_senseur-rescue:R-RESCUE-noeud_senseur R17
 U 1 1 58DBF562
 P 2950 2350
@@
 $EndComp
 $Comp
-L R R16
+L noeud_senseur-rescue:R-RESCUE-noeud_senseur R16
 U 1 1 58DBF60A
 P 2950 1750
@@
 $EndComp
 $Comp
-L R R15
+L noeud_senseur-rescue:R-RESCUE-noeud_senseur R15
 U 1 1 58DBF63E
 P 2400 1775
@@
 $EndComp
 $Comp
-L +3.3V #PWR52
+L noeud_senseur-rescue:+3.3V-RESCUE-noeud_senseur #PWR52
 U 1 1 58DBFD32
 P 2950 1375
@@
 $EndComp
 $Comp
-L GND #PWR51
+L noeud_senseur-rescue:GND-RESCUE-noeud_senseur #PWR51
 U 1 1 58DBFD9A
 P 2575 2600
@@
 $EndComp
 $Comp
-L CP C9
+L noeud_senseur-rescue:CP-RESCUE-noeud_senseur C9
 U 1 1 58DC0245
 P 2575 2350
@@
 Connection ~ 2950 2050
 $Comp
-L GND #PWR53
+L noeud_senseur-rescue:GND-RESCUE-noeud_senseur #PWR53
 U 1 1 58DC135A
 P 2950 2600
@@
 Burden Resistor\n30A -> 100 ohm, 3.3V\n100A -> 18 ohm, 3.3V - 33 ohm, 5V
 $Comp
-L R R21
+L noeud_senseur-rescue:R-RESCUE-noeud_senseur R21
 U 1 1 58DC40AC
 P 6475 2350
@@
 $EndComp
 $Comp
-L R R20
+L noeud_senseur-rescue:R-RESCUE-noeud_senseur R20
 U 1 1 58DC40B2
 P 6475 1750
@@
 $EndComp
 $Comp
-L R R19
+L noeud_senseur-rescue:R-RESCUE-noeud_senseur R19
 U 1 1 58DC40B8
 P 5925 1775
@@
 $EndComp
 $Comp
-L +3.3V #PWR55
+L noeud_senseur-rescue:+3.3V-RESCUE-noeud_senseur #PWR55
 U 1 1 58DC40BE
 P 6475 1375
@@
 $EndComp
 $Comp
-L GND #PWR54
+L noeud_senseur-rescue:GND-RESCUE-noeud_senseur #PWR54
 U 1 1 58DC40C4
 P 6100 2600
@@
 $EndComp
 $Comp
-L CP C10
+L noeud_senseur-rescue:CP-RESCUE-noeud_senseur C10
 U 1 1 58DC40CA
 P 6100 2350
@@
 Connection ~ 6475 2050
 $Comp
-L GND #PWR56
+L noeud_senseur-rescue:GND-RESCUE-noeud_senseur #PWR56
 U 1 1 58DC40D8
 P 6475 2600
@@
 Connection ~ 5925 1550
 $Comp
-L R R18
+L noeud_senseur-rescue:R-RESCUE-noeud_senseur R18
 U 1 1 58DC43F4
 P 5300 1550
@@
 VT_OUT
 $Comp
-L JACK_TRS_3PINS CT-1
+L jfng:JACK_TRS_3PINS CT-1
 U 1 1 58E21616
 P 1175 1850
@@
 NoConn ~ 1575 1650
 $Comp
-L Barrel_Jack VT-1
+L jfng:Barrel_Jack VT-1
 U 1 1 5939738C
 P 4700 1650
