File: Kicad/SPI.sch (KiCad schematic (older format))
At the start: 11 parts, among them U4 SN65HVD232Q, U5 MCP2515, Y1 16MHz

Commit message: Mise a jour du 6 juillet 2017
Parts:
- added R23: 10k, Resistors_SMD:R_0805_HandSoldering, symbol R
- C12: value 0.1uF -> 1uF
Connections:
- net +3V3: now also C1.2, R23.1; no longer C1.1
- net GND: now also C1.1; no longer C1.2
- net at U5.17 (~RESET): now also R23.2
- no-connect marks 9 -> 8
Other:
- moved on the sheet: C1, C6
Changed lines of the file:
@@
 EESchema Schematic File Version 2
+LIBS:noeud_senseur-rescue
 LIBS:power
 LIBS:device
@@
 EELAYER 26 0
 EELAYER END
-$Descr A4 11693 8268
+$Descr USLetter 11000 8500
 encoding utf-8
 Sheet 2 5
-Title ""
-Date ""
-Rev ""
+Title "SPI"
+Date "2017-06-06"
+Rev "1.1"
 Comp ""
 Comment1 ""
@@
 $EndDescr
 $Comp
-L +3.3V #PWR014
+L +3.3V #PWR16
 U 1 1 58C15170
 P 4875 4275
-F 0 "#PWR014" H 1350 -1200 50  0001 C CNN
+F 0 "#PWR16" H 1350 -1200 50  0001 C CNN
 F 1 "+3.3V" H 5000 4300 50  0000 C CNN
 F 2 "" H 1350 -1050 50  0001 C CNN
@@
 	-1   0    0    -1
 $EndComp
-Wire Wire Line
-	6175 4975 5925 4975
-Wire Wire Line
-	6175 5075 5150 5075
-Wire Wire Line
-	5925 5175 6175 5175
-Wire Wire Line
-	4875 5275 6175 5275
-Wire Wire Line
-	6175 5375 5925 5375
-Wire Wire Line
-	6175 5475 5925 5475
-Wire Wire Line
-	5150 5075 5150 5850
-$Comp
-L GND #PWR015
+$Comp
+L GND #PWR17
 U 1 1 58C15188
 P 5150 5850
-F 0 "#PWR015" H 5200 5900 50  0001 C CNN
+F 0 "#PWR17" H 5200 5900 50  0001 C CNN
 F 1 "GND" H 5155 5677 50  0000 C CNN
 F 2 "" H -2750 3750 50  0001 C CNN
@@
 	1    0    0    -1
 $EndComp
-Wire Wire Line
-	4875 4275 4875 5275
 $Comp
 L C_Small C4
@@
 	1    0    0    -1
 $EndComp
-Wire Wire Line
-	4875 4350 5900 4350
-Wire Wire Line
-	5475 4350 5475 4375
-Connection ~ 4875 4350
-Wire Wire Line
-	5100 4375 5100 4350
-Connection ~ 5100 4350
-Wire Wire Line
-	5100 4575 5900 4575
-Wire Wire Line
-	5275 4575 5275 4650
-Connection ~ 5275 4575
-$Comp
-L GND #PWR016
+$Comp
+L GND #PWR18
 U 1 1 58C151B6
 P 5275 4650
-F 0 "#PWR016" H -2750 3375 50  0001 C CNN
+F 0 "#PWR18" H -2750 3375 50  0001 C CNN
 F 1 "GND" H 5280 4477 50  0000 C CNN
 F 2 "" H -2750 3625 50  0001 C CNN
@@
 $EndComp
 $Comp
-L +3.3V #PWR018
+L +3.3V #PWR20
 U 1 1 58C161E4
-P 7150 2150
-F 0 "#PWR018" H 7200 2200 50  0001 C CNN
-F 1 "+3.3V" H 7165 2323 50  0000 C CNN
-F 2 "" H -625 -725 50  0001 C CNN
-F 3 "" H -625 -725 50  0001 C CNN
-	1    7150 2150
-	1    0    0    -1
-$EndComp
-NoConn ~ 7025 2450
+P 7150 1800
+F 0 "#PWR20" H 7200 1850 50  0001 C CNN
+F 1 "+3.3V" H 7165 1973 50  0000 C CNN
+F 2 "" H -625 -1075 50  0001 C CNN
+F 3 "" H -625 -1075 50  0001 C CNN
+	1    7150 1800
+	1    0    0    -1
+$EndComp
 NoConn ~ 7025 3050
 NoConn ~ 7025 3150
@@
 NoConn ~ 5725 2850
 $Comp
-L GND #PWR019
+L GND #PWR19
 U 1 1 58C161F0
 P 5725 3150
-F 0 "#PWR019" H 5775 3200 50  0001 C CNN
+F 0 "#PWR19" H 5775 3200 50  0001 C CNN
 F 1 "GND" H 5730 2977 50  0000 C CNN
 F 2 "" H -500 -700 50  0001 C CNN
@@
 $EndComp
 NoConn ~ 5725 2550
-$Comp
-L SN65HVD232Q U4
-U 1 1 58C161F7
-P 4075 2550
-F 0 "U4" H 4400 2900 50  0000 C CNN
-F 1 "SN65HVD232Q" H 3775 2175 50  0000 C CNN
-F 2 "Housings_SOIC:SOIC-8_3.9x4.9mm_Pitch1.27mm" H -625 -1325 50  0001 C CIN
-F 3 "" H -625 -825 50  0001 C CNN
-	1    4075 2550
-	-1   0    0    -1
-$EndComp
 $Comp
 L Crystal_Small Y1
@@
 $EndComp
 $Comp
-L GND #PWR020
+L GND #PWR15
 U 1 1 58C16216
 P 4825 3425
-F 0 "#PWR020" H -500 -950 50  0001 C CNN
+F 0 "#PWR15" H -500 -950 50  0001 C CNN
 F 1 "GND" H 4830 3252 50  0000 C CNN
 F 2 "" H -500 -700 50  0001 C CNN
@@
 $EndComp
 $Comp
-L +3.3V #PWR021
+L +3.3V #PWR12
 U 1 1 58C1621C
 P 4075 1175
-F 0 "#PWR021" H 4125 1225 50  0001 C CNN
+F 0 "#PWR12" H 4125 1225 50  0001 C CNN
 F 1 "+3.3V" H 4090 1348 50  0000 C CNN
 F 2 "" H -3700 -1700 50  0001 C CNN
@@
 $EndComp
 $Comp
-L GND #PWR022
+L GND #PWR13
 U 1 1 58C16222
 P 4075 3025
-F 0 "#PWR022" H 4125 3075 50  0001 C CNN
+F 0 "#PWR13" H 4125 3075 50  0001 C CNN
 F 1 "GND" H 4080 2852 50  0000 C CNN
 F 2 "" H -2150 -825 50  0001 C CNN
@@
 L C_Small C6
 U 1 1 58C1623F
-P 8500 2425
-F 0 "C6" H 8592 2471 50  0000 L CNN
-F 1 "0.1uF" H 8592 2380 50  0000 L CNN
-F 2 "Capacitors_SMD:C_0805_HandSoldering" H 2525 -4350 50  0001 C CNN
-F 3 "" H 2525 -4350 50  0001 C CNN
-	1    8500 2425
-	1    0    0    -1
-$EndComp
-$Comp
-L GND #PWR023
+P 7350 1950
+F 0 "C6" V 7450 1900 50  0000 L CNN
+F 1 "0.1uF" V 7225 1850 50  0000 L CNN
+F 2 "Capacitors_SMD:C_0805_HandSoldering" H 1375 -4825 50  0001 C CNN
+F 3 "" H 1375 -4825 50  0001 C CNN
+	1    7350 1950
+	0    -1   -1   0
+$EndComp
+$Comp
+L GND #PWR21
 U 1 1 58C16246
-P 8500 2650
-F 0 "#PWR023" H 2775 -675 50  0001 C CNN
-F 1 "GND" H 8505 2477 50  0000 C CNN
-F 2 "" H 2775 -425 50  0001 C CNN
-F 3 "" H 2775 -425 50  0001 C CNN
-	1    8500 2650
+P 7525 2075
+F 0 "#PWR21" H 1800 -1250 50  0001 C CNN
+F 1 "GND" H 7530 1902 50  0000 C CNN
+F 2 "" H 1800 -1000 50  0001 C CNN
+F 3 "" H 1800 -1000 50  0001 C CNN
+	1    7525 2075
 	1    0    0    -1
 $EndComp
@@
 L C_Small C1
 U 1 1 58C1624C
-P 4500 1575
-F 0 "C1" H 4592 1621 50  0000 L CNN
-F 1 "0.1uF" H 4592 1530 50  0000 L CNN
-F 2 "Capacitors_SMD:C_0805_HandSoldering" H -1475 -5200 50  0001 C CNN
-F 3 "" H -1475 -5200 50  0001 C CNN
-	1    4500 1575
-	1    0    0    -1
-$EndComp
-$Comp
-L GND #PWR024
+P 4400 1300
+F 0 "C1" V 4300 1250 50  0000 L CNN
+F 1 "0.1uF" V 4525 1225 50  0000 L CNN
+F 2 "Capacitors_SMD:C_0805_HandSoldering" H -1575 -5475 50  0001 C CNN
+F 3 "" H -1575 -5475 50  0001 C CNN
+	1    4400 1300
+	0    1    1    0
+$EndComp
+$Comp
+L GND #PWR14
 U 1 1 58C16253
-P 4500 1775
-F 0 "#PWR024" H 4550 1825 50  0001 C CNN
-F 1 "GND" H 4505 1602 50  0000 C CNN
-F 2 "" H -1725 -2075 50  0001 C CNN
-F 3 "" H -1725 -2075 50  0001 C CNN
-	1    4500 1775
-	1    0    0    -1
-$EndComp
-Wire Wire Line
-	4500 1675 4500 1775
-Connection ~ 4075 1300
-Wire Wire Line
-	4500 1300 4075 1300
-Wire Wire Line
-	4500 1475 4500 1300
-Wire Wire Line
-	8500 2525 8500 2650
-Connection ~ 7150 2250
-Wire Wire Line
-	8500 2250 7150 2250
-Wire Wire Line
-	8500 2325 8500 2250
-Wire Wire Line
-	3475 2650 3575 2650
-Wire Wire Line
-	3475 2450 3575 2450
-Wire Wire Line
-	4075 1175 4075 2150
-Wire Wire Line
-	4075 3025 4075 2950
-Connection ~ 4825 3275
-Wire Wire Line
-	4950 3275 4825 3275
-Wire Wire Line
-	4825 2775 4825 3425
-Wire Wire Line
-	4950 2775 4825 2775
-Connection ~ 5225 3275
-Wire Wire Line
-	5225 3275 5225 3125
-Wire Wire Line
-	5150 3275 5550 3275
-Connection ~ 5225 2775
-Wire Wire Line
-	5150 2775 5550 2775
-Wire Wire Line
-	5225 2775 5225 2925
-Wire Wire Line
-	5550 3275 5550 3050
-Wire Wire Line
-	5550 3050 5725 3050
-Wire Wire Line
-	5550 2775 5550 2950
-Wire Wire Line
-	5550 2950 5725 2950
-Wire Wire Line
-	7150 2150 7150 2350
-Wire Wire Line
-	7150 2350 7025 2350
-Wire Wire Line
-	5725 2450 4575 2450
-Wire Wire Line
-	5725 2350 4575 2350
+P 4650 1425
+F 0 "#PWR14" H 4700 1475 50  0001 C CNN
+F 1 "GND" H 4655 1252 50  0000 C CNN
+F 2 "" H -1575 -2425 50  0001 C CNN
+F 3 "" H -1575 -2425 50  0001 C CNN
+	1    4650 1425
+	1    0    0    -1
+$EndComp
 Text HLabel 3475 2450 0    60   BiDi ~ 0
 CAN+
@@
 P 5900 4475
 F 0 "C12" H 5992 4521 50  0000 L CNN
-F 1 "0.1uF" H 5992 4430 50  0000 L CNN
+F 1 "1uF" H 5992 4430 50  0000 L CNN
 F 2 "Capacitors_SMD:C_0805_HandSoldering" H -75 -2300 50  0001 C CNN
 F 3 "" H -75 -2300 50  0001 C CNN
@@
 	1    0    0    -1
 $EndComp
-Connection ~ 5475 4575
-Wire Wire Line
-	5900 4350 5900 4375
-Connection ~ 5475 4350
-Text Label 4950 2350 0    60   ~ 0
+Text Label 4650 2350 0    60   ~ 0
 TXC
-Text Label 4950 2450 0    60   ~ 0
+Text Label 4650 2450 0    60   ~ 0
 RXC
 $Comp
@@
 	1    0    0    1
 $EndComp
+$Comp
+L SN65HVD232Q U4
+U 1 1 5938C27E
+P 4075 2550
+F 0 "U4" H 4400 2900 50  0000 C CNN
+F 1 "SN65HVD232Q" H 3750 2175 50  0000 C CNN
+F 2 "Housings_SOIC:SOIC-8_3.9x4.9mm_Pitch1.27mm" H 4075 2050 50  0001 C CIN
+F 3 "" H 4075 2550 50  0001 C CNN
+	1    4075 2550
+	-1   0    0    -1
+$EndComp
+Wire Wire Line
+	6175 4975 5925 4975
+Wire Wire Line
+	6175 5075 5150 5075
+Wire Wire Line
+	5925 5175 6175 5175
+Wire Wire Line
+	4875 5275 6175 5275
+Wire Wire Line
+	6175 5375 5925 5375
+Wire Wire Line
+	6175 5475 5925 5475
+Wire Wire Line
+	5150 5075 5150 5850
+Wire Wire Line
+	4875 4275 4875 5275
+Wire Wire Line
+	4875 4350 5900 4350
+Wire Wire Line
+	5475 4350 5475 4375
+Connection ~ 4875 4350
+Wire Wire Line
+	5100 4375 5100 4350
+Connection ~ 5100 4350
+Wire Wire Line
+	5100 4575 5900 4575
+Wire Wire Line
+	5275 4575 5275 4650
+Connection ~ 5275 4575
+Connection ~ 4075 1300
+Wire Wire Line
+	4300 1300 4075 1300
+Wire Wire Line
+	7525 1950 7525 2075
+Wire Wire Line
+	3475 2650 3575 2650
+Wire Wire Line
+	3475 2450 3575 2450
+Wire Wire Line
+	4075 1175 4075 2150
+Wire Wire Line
+	4075 3025 4075 2950
+Connection ~ 4825 3275
+Wire Wire Line
+	4950 3275 4825 3275
+Wire Wire Line
+	4825 2775 4825 3425
+Wire Wire Line
+	4950 2775 4825 2775
+Connection ~ 5225 3275
+Wire Wire Line
+	5225 3275 5225 3125
+Wire Wire Line
+	5150 3275 5550 3275
+Connection ~ 5225 2775
+Wire Wire Line
+	5150 2775 5550 2775
+Wire Wire Line
+	5225 2775 5225 2925
+Wire Wire Line
+	5550 3275 5550 3050
+Wire Wire Line
+	5550 3050 5725 3050
+Wire Wire Line
+	5550 2775 5550 2950
+Wire Wire Line
+	5550 2950 5725 2950
+Wire Wire Line
+	7150 1800 7150 2350
+Wire Wire Line
+	7150 2350 7025 2350
+Wire Wire Line
+	5725 2450 4575 2450
+Wire Wire Line
+	5725 2350 4575 2350
+Connection ~ 5475 4575
+Wire Wire Line
+	5900 4350 5900 4375
+Connection ~ 5475 4350
+Wire Wire Line
+	7025 2450 7775 2450
+Wire Wire Line
+	7775 2450 7775 2250
+Wire Wire Line
+	7250 1950 7150 1950
+Connection ~ 7150 1950
+Wire Wire Line
+	7450 1950 7525 1950
+$Comp
+L R R23
+U 1 1 5938D9DF
+P 7775 2100
+F 0 "R23" H 7845 2146 50  0000 L CNN
+F 1 "10k" H 7845 2055 50  0000 L CNN
+F 2 "Resistors_SMD:R_0805_HandSoldering" V 7705 2100 50  0001 C CNN
+F 3 "" H 7775 2100 50  0001 C CNN
+	1    7775 2100
+	1    0    0    -1
+$EndComp
+Wire Wire Line
+	7775 1950 7775 1800
+$Comp
+L +3.3V #PWR22
+U 1 1 5938DB22
+P 7775 1800
+F 0 "#PWR22" H 7825 1850 50  0001 C CNN
+F 1 "+3.3V" H 7790 1973 50  0000 C CNN
+F 2 "" H 0   -1075 50  0001 C CNN
+F 3 "" H 0   -1075 50  0001 C CNN
+	1    7775 1800
+	1    0    0    -1
+$EndComp
+Wire Wire Line
+	4650 1425 4650 1300
+Wire Wire Line
+	4650 1300 4500 1300
 $EndSCHEMATC

Commit message: Recompilation des applications.
Parts:
- C1, C12, C2, C3, C4, C5, C6: symbol C_Small -> noeud_senseur-rescue:C_Small-RESCUE-noeud_senseur
- R23: symbol R -> noeud_senseur-rescue:R-RESCUE-noeud_senseur
- U4: symbol SN65HVD232Q -> jfng:SN65HVD232Q
- U5: symbol MCP2515 -> jfng:MCP2515
- Y1: symbol Crystal_Small -> noeud_senseur-rescue:Crystal_Small-RESCUE-noeud_senseur
- uSD-1: symbol Micro_SD_Card_no_shield -> jfng:Micro_SD_Card_no_shield
Changed lines of the file:
@@
-EESchema Schematic File Version 2
-LIBS:noeud_senseur-rescue
-LIBS:power
-LIBS:device
-LIBS:transistors
-LIBS:conn
-LIBS:linear
-LIBS:regul
-LIBS:74xx
-LIBS:cmos4000
-LIBS:adc-dac
-LIBS:memory
-LIBS:xilinx
-LIBS:microcontrollers
-LIBS:dsp
-LIBS:microchip
-LIBS:analog_switches
-LIBS:motorola
-LIBS:texas
-LIBS:intel
-LIBS:audio
-LIBS:interface
-LIBS:digital-audio
-LIBS:philips
-LIBS:display
-LIBS:cypress
-LIBS:siliconi
-LIBS:opto
-LIBS:atmel
-LIBS:contrib
-LIBS:valves
-LIBS:jfng
+EESchema Schematic File Version 4
 LIBS:noeud_senseur-cache
 EELAYER 26 0
@@
 $EndDescr
 $Comp
-L +3.3V #PWR16
+L noeud_senseur-rescue:+3.3V-RESCUE-noeud_senseur #PWR16
 U 1 1 58C15170
 P 4875 4275
@@
 $EndComp
 $Comp
-L GND #PWR17
+L noeud_senseur-rescue:GND-RESCUE-noeud_senseur #PWR17
 U 1 1 58C15188
 P 5150 5850
@@
 $EndComp
 $Comp
-L C_Small C4
+L noeud_senseur-rescue:C_Small-RESCUE-noeud_senseur C4
 U 1 1 58C151A0
 P 5100 4475
@@
 $EndComp
 $Comp
-L C_Small C5
+L noeud_senseur-rescue:C_Small-RESCUE-noeud_senseur C5
 U 1 1 58C151A7
 P 5475 4475
@@
 $EndComp
 $Comp
-L GND #PWR18
+L noeud_senseur-rescue:GND-RESCUE-noeud_senseur #PWR18
 U 1 1 58C151B6
 P 5275 4650
@@
 $EndComp
 $Comp
-L MCP2515 U5
+L jfng:MCP2515 U5
 U 1 1 58C161DD
 P 6375 2750
@@
 $EndComp
 $Comp
-L +3.3V #PWR20
+L noeud_senseur-rescue:+3.3V-RESCUE-noeud_senseur #PWR20
 U 1 1 58C161E4
 P 7150 1800
@@
 NoConn ~ 5725 2850
 $Comp
-L GND #PWR19
+L noeud_senseur-rescue:GND-RESCUE-noeud_senseur #PWR19
 U 1 1 58C161F0
 P 5725 3150
@@
 NoConn ~ 5725 2550
 $Comp
-L Crystal_Small Y1
+L noeud_senseur-rescue:Crystal_Small-RESCUE-noeud_senseur Y1
 U 1 1 58C16201
 P 5225 3025
@@
 $EndComp
 $Comp
-L C_Small C2
+L noeud_senseur-rescue:C_Small-RESCUE-noeud_senseur C2
 U 1 1 58C16208
 P 5050 2775
@@
 $EndComp
 $Comp
-L C_Small C3
+L noeud_senseur-rescue:C_Small-RESCUE-noeud_senseur C3
 U 1 1 58C1620F
 P 5050 3275
@@
 $EndComp
 $Comp
-L GND #PWR15
+L noeud_senseur-rescue:GND-RESCUE-noeud_senseur #PWR15
 U 1 1 58C16216
 P 4825 3425
@@
 $EndComp
 $Comp
-L +3.3V #PWR12
+L noeud_senseur-rescue:+3.3V-RESCUE-noeud_senseur #PWR12
 U 1 1 58C1621C
 P 4075 1175
@@
 $EndComp
 $Comp
-L GND #PWR13
+L noeud_senseur-rescue:GND-RESCUE-noeud_senseur #PWR13
 U 1 1 58C16222
 P 4075 3025
@@
 $EndComp
 $Comp
-L C_Small C6
+L noeud_senseur-rescue:C_Small-RESCUE-noeud_senseur C6
 U 1 1 58C1623F
 P 7350 1950
@@
 $EndComp
 $Comp
-L GND #PWR21
+L noeud_senseur-rescue:GND-RESCUE-noeud_senseur #PWR21
 U 1 1 58C16246
 P 7525 2075
@@
 $EndComp
 $Comp
-L C_Small C1
+L noeud_senseur-rescue:C_Small-RESCUE-noeud_senseur C1
 U 1 1 58C1624C
 P 4400 1300
@@
 $EndComp
 $Comp
-L GND #PWR14
+L noeud_senseur-rescue:GND-RESCUE-noeud_senseur #PWR14
 U 1 1 58C16253
 P 4650 1425
@@
 NoConn ~ 6175 5575
 $Comp
-L C_Small C12
+L noeud_senseur-rescue:C_Small-RESCUE-noeud_senseur C12
 U 1 1 58EFF980
 P 5900 4475
@@
 RXC
 $Comp
-L Micro_SD_Card_no_shield uSD-1
+L jfng:Micro_SD_Card_no_shield uSD-1
 U 1 1 5900282A
 P 7075 5275
@@
 $EndComp
 $Comp
-L SN65HVD232Q U4
+L jfng:SN65HVD232Q U4
 U 1 1 5938C27E
 P 4075 2550
@@
 	7450 1950 7525 1950
 $Comp
-L R R23
+L noeud_senseur-rescue:R-RESCUE-noeud_senseur R23
 U 1 1 5938D9DF
 P 7775 2100
@@
 	7775 1950 7775 1800
 $Comp
-L +3.3V #PWR22
+L noeud_senseur-rescue:+3.3V-RESCUE-noeud_senseur #PWR22
 U 1 1 5938DB22
 P 7775 1800
