File: Kicad/noeud_senseur.sch (KiCad schematic (older format))
At the start: 14 parts, among them Q1 DMG1012UW, Q2 DMG1012UW, Q3 LP0701_SGD, U2 DS18B20

Commit message: Mise a jour du 6 juillet 2017
Parts:
- added JP1: Jumper, Pin_Headers:Pin_Header_Straight_1x02_Pitch2.54mm, symbol Jumper
- Adafruit_Feather-1: symbol FEATHER_MO_LORA -> FEATHER_MO_LORA-RESCUE-noeud_senseur
Connections:
- wire segments 84 -> 87
Other:
- moved on the sheet: S1
Changed lines of the file:
@@
 EESchema Schematic File Version 2
+LIBS:noeud_senseur-rescue
 LIBS:power
 LIBS:device
@@
 encoding utf-8
 Sheet 1 5
-Title ""
-Date "2017-02-23"
-Rev ""
+Title "Noeud Senseur"
+Date "2017-06-06"
+Rev "1.1"
 Comp ""
 Comment1 ""
@@
 SDA
 $Comp
-L +3.3V #PWR01
+L +3.3V #PWR8
 U 1 1 588F82DF
 P 4725 2375
-F 0 "#PWR01" H -575 -725 50  0001 C CNN
+F 0 "#PWR8" H -575 -725 50  0001 C CNN
 F 1 "+3.3V" H 4740 2548 50  0000 C CNN
 F 2 "" H -575 -575 50  0001 C CNN
@@
 $EndComp
 $Comp
-L +3.3V #PWR02
+L +3.3V #PWR3
 U 1 1 588FA539
 P 1875 1525
-F 0 "#PWR02" H -3425 -1575 50  0001 C CNN
+F 0 "#PWR3" H -3425 -1575 50  0001 C CNN
 F 1 "+3.3V" H 1890 1698 50  0000 C CNN
 F 2 "" H -3425 -1425 50  0001 C CNN
@@
 A2
 $Comp
-L GND #PWR03
+L GND #PWR1
 U 1 1 588FEF8A
 P 1325 1975
-F 0 "#PWR03" H -4400 -1350 50  0001 C CNN
+F 0 "#PWR1" H -4400 -1350 50  0001 C CNN
 F 1 "GND" H 1330 1802 50  0000 C CNN
 F 2 "" H -4400 -1100 50  0001 C CNN
@@
 Text Label 1750 2200 0    60   ~ 0
 A3
-$Comp
-L DS18B20 U2
-U 1 1 5890D83B
-P 5825 5775
-F 0 "U2" H 5675 6025 50  0000 L CNN
-F 1 "DS18B20" H 5650 5500 50  0000 L CNN
-F 2 "TO_SOT_Packages_THT:TO-92_Inline_Wide" H 2050 -500 50  0001 C CNN
-F 3 "" H 2050 -500 50  0001 C CNN
-	1    5825 5775
-	1    0    0    -1
-$EndComp
 Text Label 4125 2800 2    60   ~ 0
 1_WIRE_IO
@@
 1_WIRE_IO
 $Comp
-L +3.3V #PWR04
+L +3.3V #PWR9
 U 1 1 5890E20D
 P 5050 5325
-F 0 "#PWR04" H -250 2225 50  0001 C CNN
+F 0 "#PWR9" H -250 2225 50  0001 C CNN
 F 1 "+3.3V" H 5065 5498 50  0000 C CNN
 F 2 "" H -250 2375 50  0001 C CNN
@@
 $EndComp
 $Comp
-L GND #PWR05
+L GND #PWR10
 U 1 1 5890E24B
 P 5050 5950
-F 0 "#PWR05" H -675 2625 50  0001 C CNN
+F 0 "#PWR10" H -675 2625 50  0001 C CNN
 F 1 "GND" H 5055 5777 50  0000 C CNN
 F 2 "" H -675 2875 50  0001 C CNN
@@
 A5
 $Comp
-L GND #PWR06
+L GND #PWR5
 U 1 1 58A6E58C
 P 2125 5925
-F 0 "#PWR06" H -3600 2600 50  0001 C CNN
+F 0 "#PWR5" H -3600 2600 50  0001 C CNN
 F 1 "GND" H 2130 5752 50  0000 C CNN
 F 2 "" H -3600 2850 50  0001 C CNN
@@
 $EndComp
 $Comp
-L +3.3V #PWR07
+L +3.3V #PWR4
 U 1 1 58A718EA
 P 2125 4625
-F 0 "#PWR07" H -3175 1525 50  0001 C CNN
+F 0 "#PWR4" H -3175 1525 50  0001 C CNN
 F 1 "+3.3V" H 2140 4798 50  0000 C CNN
 F 2 "" H -3175 1675 50  0001 C CNN
@@
 $EndComp
 $Comp
-L GND #PWR08
+L GND #PWR7
 U 1 1 58A74946
 P 3300 5925
-F 0 "#PWR08" H -2425 2600 50  0001 C CNN
+F 0 "#PWR7" H -2425 2600 50  0001 C CNN
 F 1 "GND" H 3305 5752 50  0000 C CNN
 F 2 "" H -2425 2850 50  0001 C CNN
@@
 $EndComp
 $Comp
-L +3.3V #PWR09
+L +3.3V #PWR6
 U 1 1 58A7495A
 P 3300 4625
-F 0 "#PWR09" H -2000 1525 50  0001 C CNN
+F 0 "#PWR6" H -2000 1525 50  0001 C CNN
 F 1 "+3.3V" H 3315 4798 50  0000 C CNN
 F 2 "" H -2000 1675 50  0001 C CNN
@@
 $EndComp
 $Comp
-L +3.3V #PWR010
+L +3.3V #PWR2
 U 1 1 58A74E2F
 P 1625 1525
-F 0 "#PWR010" H -3675 -1575 50  0001 C CNN
+F 0 "#PWR2" H -3675 -1575 50  0001 C CNN
 F 1 "+3.3V" H 1640 1698 50  0000 C CNN
 F 2 "" H -3675 -1425 50  0001 C CNN
@@
 NoConn ~ 3450 1900
 $Comp
-L FEATHER_MO_LORA Adafruit_Feather-1
+L FEATHER_MO_LORA-RESCUE-noeud_senseur Adafruit_Feather-1
 U 1 1 58A7C9E5
 P 2800 2400
@@
 $EndComp
 $Comp
-L PWR_FLAG #FLG011
+L PWR_FLAG #FLG2
 U 1 1 58A85600
 P 4400 1425
-F 0 "#FLG011" H 0   -3175 50  0001 C CNN
+F 0 "#FLG2" H 0   -3175 50  0001 C CNN
 F 1 "PWR_FLAG" H 4400 1599 50  0000 C CNN
 F 2 "" H 0   -3250 50  0001 C CNN
@@
 $EndComp
 $Comp
-L PWR_FLAG #FLG012
+L PWR_FLAG #FLG1
 U 1 1 58A87270
 P 1325 1650
-F 0 "#FLG012" H 225 -3225 50  0001 C CNN
+F 0 "#FLG1" H 225 -3225 50  0001 C CNN
 F 1 "PWR_FLAG" H 1325 1824 50  0000 C CNN
 F 2 "" H 225 -3300 50  0001 C CNN
@@
 L ORD211-1015 S1
 U 1 1 58AD8EEB
-P 5375 1900
-F 0 "S1" V 5322 1988 60  0000 L CNN
-F 1 "ORD211-1015" V 5428 1988 60  0000 L CNN
-F 2 "Pin_Headers:Pin_Header_Straight_1x02_Pitch2.54mm" H 1225 -2150 60  0001 C CNN
-F 3 "" H 1225 -2150 60  0001 C CNN
-	1    5375 1900
+P 5775 1900
+F 0 "S1" V 5722 1988 60  0000 L CNN
+F 1 "ORD211-1015" V 5828 1988 60  0000 L CNN
+F 2 "Pin_Headers:Pin_Header_Straight_1x02_Pitch2.54mm" H 1625 -2150 60  0001 C CNN
+F 3 "" H 1625 -2150 60  0001 C CNN
+	1    5775 1900
 	0    1    1    0
 $EndComp
 $Comp
-L GND #PWR013
+L GND #PWR11
 U 1 1 58AE33ED
-P 5375 2175
-F 0 "#PWR013" H -350 -1150 50  0001 C CNN
-F 1 "GND" H 5380 2002 50  0000 C CNN
-F 2 "" H -350 -900 50  0001 C CNN
-F 3 "" H -350 -900 50  0001 C CNN
-	1    5375 2175
+P 5775 2175
+F 0 "#PWR11" H 50  -1150 50  0001 C CNN
+F 1 "GND" H 5780 2002 50  0000 C CNN
+F 2 "" H 50  -900 50  0001 C CNN
+F 3 "" H 50  -900 50  0001 C CNN
+	1    5775 2175
 	1    0    0    -1
 $EndComp
@@
 	0    1    1    0
 $EndComp
-Connection ~ 5375 1625
-Wire Wire Line
-	5375 1700 5375 1625
 Connection ~ 4975 1625
 Wire Wire Line
@@
 	4400 1500 4400 1425
 Wire Wire Line
-	3450 2700 4125 2700
+	3450 2700 4475 2700
 Wire Wire Line
 	3450 2300 4125 2300
@@
 	3450 2900 4725 2900
 Wire Wire Line
-	5375 2175 5375 2100
+	5775 2175 5775 2100
 $Sheet
 S 6575 2350 1175 850
@@
 Text Label 8025 4100 0    60   ~ 0
 1_WIRE_IO
+$Comp
+L DS18B20 U2
+U 1 1 593A33A5
+P 5825 5775
+F 0 "U2" H 6052 5821 50  0000 L CNN
+F 1 "DS18B20" H 6052 5730 50  0000 L CNN
+F 2 "TO_SOT_Packages_THT:TO-92_Inline_Wide" H 5675 6025 50  0001 C CNN
+F 3 "" H 5675 6025 50  0001 C CNN
+	1    5825 5775
+	1    0    0    -1
+$EndComp
+$Comp
+L Jumper JP1
+U 1 1 5949FBE4
+P 5100 2050
+F 0 "JP1" H 5100 2314 50  0000 C CNN
+F 1 "Jumper" H 5100 2223 50  0000 C CNN
+F 2 "Pin_Headers:Pin_Header_Straight_1x02_Pitch2.54mm" H 5100 2050 50  0001 C CNN
+F 3 "" H 5100 2050 50  0001 C CNN
+	1    5100 2050
+	1    0    0    -1
+$EndComp
+Wire Wire Line
+	5775 1700 5775 1625
+Connection ~ 5775 1625
+Wire Wire Line
+	5400 2050 5400 1625
+Connection ~ 5400 1625
+Wire Wire Line
+	4475 2700 4475 2050
+Wire Wire Line
+	4475 2050 4800 2050
 $EndSCHEMATC

Commit message: Recompilation des applications.
Parts:
- Adafruit_Feather-1: symbol FEATHER_MO_LORA-RESCUE-noeud_senseur -> noeud_senseur-rescue:FEATHER_MO_LORA-RESCUE-noeud_senseur
- D1, D2: symbol LED -> noeud_senseur-rescue:LED-RESCUE-noeud_senseur
- JP1: symbol Jumper -> noeud_senseur-rescue:Jumper-RESCUE-noeud_senseur
- Q1, Q2: symbol DMG1012T -> jfng:DMG1012T
- Q3: symbol Q_PMOS_SGD -> jfng:Q_PMOS_SGD
- R1, R2, R3, R4, R5, R6: symbol R -> noeud_senseur-rescue:R-RESCUE-noeud_senseur
- S1: symbol ORD211-1015 -> jfng:ORD211-1015
- U2: symbol DS18B20 -> jfng:DS18B20
Connections:
- wire segments 87 -> 96
Changed lines of the file:
@@
-EESchema Schematic File Version 2
-LIBS:noeud_senseur-rescue
-LIBS:power
-LIBS:device
-LIBS:transistors
-LIBS:conn
-LIBS:linear
-LIBS:regul
-LIBS:74xx
-LIBS:cmos4000
-LIBS:adc-dac
-LIBS:memory
-LIBS:xilinx
-LIBS:microcontrollers
-LIBS:dsp
-LIBS:microchip
-LIBS:analog_switches
-LIBS:motorola
-LIBS:texas
-LIBS:intel
-LIBS:audio
-LIBS:interface
-LIBS:digital-audio
-LIBS:philips
-LIBS:display
-LIBS:cypress
-LIBS:siliconi
-LIBS:opto
-LIBS:atmel
-LIBS:contrib
-LIBS:valves
-LIBS:jfng
+EESchema Schematic File Version 4
 LIBS:noeud_senseur-cache
 EELAYER 26 0
@@
 SDA
 $Comp
-L +3.3V #PWR8
+L noeud_senseur-rescue:+3.3V-RESCUE-noeud_senseur #PWR8
 U 1 1 588F82DF
 P 4725 2375
@@
 $EndComp
 $Comp
-L R R4
+L noeud_senseur-rescue:R-RESCUE-noeud_senseur R4
 U 1 1 588F82F4
 P 4725 2650
@@
 $EndComp
 $Comp
-L R R6
+L noeud_senseur-rescue:R-RESCUE-noeud_senseur R6
 U 1 1 588F834B
 P 5025 2650
@@
 $EndComp
 $Comp
-L +3.3V #PWR3
+L noeud_senseur-rescue:+3.3V-RESCUE-noeud_senseur #PWR3
 U 1 1 588FA539
 P 1875 1525
@@
 A2
 $Comp
-L GND #PWR1
+L noeud_senseur-rescue:GND-RESCUE-noeud_senseur #PWR1
 U 1 1 588FEF8A
 P 1325 1975
@@
 1_WIRE_IO
 $Comp
-L +3.3V #PWR9
+L noeud_senseur-rescue:+3.3V-RESCUE-noeud_senseur #PWR9
 U 1 1 5890E20D
 P 5050 5325
@@
 $EndComp
 $Comp
-L GND #PWR10
+L noeud_senseur-rescue:GND-RESCUE-noeud_senseur #PWR10
 U 1 1 5890E24B
 P 5050 5950
@@
 NoConn ~ 3450 2200
 $Comp
-L R R5
+L noeud_senseur-rescue:R-RESCUE-noeud_senseur R5
 U 1 1 58A27935
 P 4775 5550
@@
 A5
 $Comp
-L GND #PWR5
+L noeud_senseur-rescue:GND-RESCUE-noeud_senseur #PWR5
 U 1 1 58A6E58C
 P 2125 5925
@@
 $EndComp
 $Comp
-L LED D1
+L noeud_senseur-rescue:LED-RESCUE-noeud_senseur D1
 U 1 1 58A70BCB
 P 2125 5200
@@
 $EndComp
 $Comp
-L R R1
+L noeud_senseur-rescue:R-RESCUE-noeud_senseur R1
 U 1 1 58A71790
 P 2125 4825
@@
 $EndComp
 $Comp
-L +3.3V #PWR4
+L noeud_senseur-rescue:+3.3V-RESCUE-noeud_senseur #PWR4
 U 1 1 58A718EA
 P 2125 4625
@@
 LED_1
 $Comp
-L DMG1012T Q1
+L jfng:DMG1012T Q1
 U 1 1 58A736DE
 P 2025 5650
@@
 $EndComp
 $Comp
-L GND #PWR7
+L noeud_senseur-rescue:GND-RESCUE-noeud_senseur #PWR7
 U 1 1 58A74946
 P 3300 5925
@@
 $EndComp
 $Comp
-L LED D2
+L noeud_senseur-rescue:LED-RESCUE-noeud_senseur D2
 U 1 1 58A7494E
 P 3300 5200
@@
 $EndComp
 $Comp
-L R R2
+L noeud_senseur-rescue:R-RESCUE-noeud_senseur R2
 U 1 1 58A74954
 P 3300 4825
@@
 $EndComp
 $Comp
-L +3.3V #PWR6
+L noeud_senseur-rescue:+3.3V-RESCUE-noeud_senseur #PWR6
 U 1 1 58A7495A
 P 3300 4625
@@
 LED_2
 $Comp
-L DMG1012T Q2
+L jfng:DMG1012T Q2
 U 1 1 58A74964
 P 3200 5650
@@
 $EndComp
 $Comp
-L +3.3V #PWR2
+L noeud_senseur-rescue:+3.3V-RESCUE-noeud_senseur #PWR2
 U 1 1 58A74E2F
 P 1625 1525
@@
 NoConn ~ 3450 1900
 $Comp
-L FEATHER_MO_LORA-RESCUE-noeud_senseur Adafruit_Feather-1
+L noeud_senseur-rescue:FEATHER_MO_LORA-RESCUE-noeud_senseur Adafruit_Feather-1
 U 1 1 58A7C9E5
 P 2800 2400
@@
 $EndComp
 $Comp
-L PWR_FLAG #FLG2
+L noeud_senseur-rescue:PWR_FLAG-RESCUE-noeud_senseur #FLG2
 U 1 1 58A85600
 P 4400 1425
@@
 $EndComp
 $Comp
-L PWR_FLAG #FLG1
+L noeud_senseur-rescue:PWR_FLAG-RESCUE-noeud_senseur #FLG1
 U 1 1 58A87270
 P 1325 1650
@@
 $EndComp
 $Comp
-L ORD211-1015 S1
+L jfng:ORD211-1015 S1
 U 1 1 58AD8EEB
 P 5775 1900
@@
 $EndComp
 $Comp
-L GND #PWR11
+L noeud_senseur-rescue:GND-RESCUE-noeud_senseur #PWR11
 U 1 1 58AE33ED
 P 5775 2175
@@
 $EndComp
 $Comp
-L Q_PMOS_SGD Q3
+L jfng:Q_PMOS_SGD Q3
 U 1 1 58AF3766
 P 4350 1775
@@
 $EndComp
 $Comp
-L R R3
+L noeud_senseur-rescue:R-RESCUE-noeud_senseur R3
 U 1 1 58AF4304
 P 4700 1500
@@
 	4975 1500 4850 1500
 Wire Wire Line
-	4975 1500 4975 1775
+	4975 1500 4975 1625
 Wire Wire Line
 	4975 1775 4550 1775
@@
 	4250 1500 4250 1575
 Wire Wire Line
-	3525 1500 4550 1500
+	3525 1500 4250 1500
 Wire Wire Line
 	4250 2000 4250 1975
@@
 	5050 5675 5525 5675
 Wire Wire Line
-	5050 5325 5050 5675
-Wire Wire Line
-	4200 5775 5525 5775
+	5050 5325 5050 5400
+Wire Wire Line
+	4200 5775 4775 5775
 Wire Wire Line
 	3450 2800 4125 2800
@@
 	1625 1700 2100 1700
 Wire Wire Line
-	1325 1650 1325 1975
+	1325 1650 1325 1800
 Wire Wire Line
 	2100 2000 1750 2000
@@
 	5025 2450 5025 2500
 Wire Wire Line
-	4725 2375 4725 2500
+	4725 2375 4725 2450
 Wire Wire Line
 	3450 3000 5025 3000
@@
 $EndSheet
 Wire Wire Line
-	4975 1625 6600 1625
+	4975 1625 5400 1625
 Wire Wire Line
 	6600 1725 6225 1725
@@
 1_WIRE_IO
 $Comp
-L DS18B20 U2
+L jfng:DS18B20 U2
 U 1 1 593A33A5
 P 5825 5775
@@
 $EndComp
 $Comp
-L Jumper JP1
+L noeud_senseur-rescue:Jumper-RESCUE-noeud_senseur JP1
 U 1 1 5949FBE4
 P 5100 2050
@@
 Wire Wire Line
 	4475 2050 4800 2050
+Wire Wire Line
+	4975 1625 4975 1775
+Wire Wire Line
+	4250 1500 4400 1500
+Wire Wire Line
+	1325 1800 1325 1975
+Wire Wire Line
+	4400 1500 4550 1500
+Wire Wire Line
+	5050 5400 5050 5675
+Wire Wire Line
+	4775 5775 5525 5775
+Wire Wire Line
+	4725 2450 4725 2500
+Wire Wire Line
+	5775 1625 6600 1625
+Wire Wire Line
+	5400 1625 5775 1625
 $EndSCHEMATC
